File: PVDX_BatteryBoard.kicad_pcb (KiCad board)
At the start: 2 copper layers, 1 part

Commit message: connectors
Parts:
- moved REF** 6.04 mm to (64.0, 66.5)
Changed lines of the file:
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@@
 	(footprint "Thermistor_NXFT15XV103FEAB025:Thermistor_ NXFT15XV103FEAB025"
 		(layer "F.Cu")
-		(at 69.5 64)
+		(at 64 66.5)
 		(property "Reference" "REF**"
-			(at 0 -0.5 0)
+			(at -0.05 -1.8 0)
 			(unlocked yes)
 			(layer "F.SilkS")
@@
 		(attr smd)
 		(fp_rect
-			(start -2 -1)
-			(end 2.1 0.9)
+			(start -1.45 -0.7)
+			(end 1.45 0.7)
 			(stroke
 				(width 0.1)
@@
 		)
 		(fp_rect
-			(start -2.1 -1.1)
-			(end 2.2 1)
+			(start -1.55 -0.8)
+			(end 1.55 0.8)
 			(stroke
 				(width 0.05)
@@
 		)
 		(pad "1" thru_hole circle
-			(at -0.95 0)
+			(at -0.65 0)
 			(size 1 1)
 			(drill 0.5)
@@
 		)
 		(pad "2" thru_hole circle
-			(at 1.15 0)
+			(at 0.65 0)
 			(size 1 1)
 			(drill 0.5)
