File: PVDX_BatteryBoard_Board.kicad_sch (KiCad schematic)
At the start: 6 parts

Commit message: Finish battery board schematic (awaiting thermistor part no.)
Parts:
- removed BT1, BT?: Battery_Cell, symbol Device:Battery_Cell
- removed C1: C, symbol Device:C
- removed Rt_1: 16.121k, symbol Device:R_US
- removed Rt_2: 5.993k, symbol Device:R_US
- removed TH1: Thermistor_NTC_US, Thermistor_NXFT15XV103FEAB025:Thermistor_ NXFT15XV103FEAB025, symbol Device:Thermistor_NTC_US
Other:
- note removed: "route to some sort of connector (batt_out)"
