File: PVDX_BatteryBoard_Heater.kicad_sch (KiCad schematic)
At the start: 7 parts, among them Q3 PMOS, Q4 NMOS

Commit message: Finish battery board schematic (awaiting thermistor part no.)
Parts:
- added Q5: NMOS, symbol Simulation_SPICE:NMOS
- added Q6: PMOS, symbol Simulation_SPICE:PMOS
- added R10, R6, R7: 10k, symbol Device:R_US
- added R8, R9: Heater, symbol Device:Heater
Connections:
- net GND: now also Q5.3 (S), R10.2, R6.2, R8.2, R9.2
- net +5V renamed CHG_OUT
- net CHG_OUT: now also Q6.1 (D), R7.1
- new net: Q5.1 (D), Q6.2 (G), R7.2
- new net: Q6.3 (S), R10.1, R8.1, R9.1
- new net HEATER_ON_2: Q5.2 (G), R6.1

Commit message: Add thermistor & MOSFET parts/values
Parts:
- removed Q3, Q6: PMOS, symbol Simulation_SPICE:PMOS
- removed Q4, Q5: NMOS, symbol Simulation_SPICE:NMOS
- added Q1, Q2: DMC2053UVT, Package_TO_SOT_SMD:TSOT-23-6, symbol Transistor_FET:DMC2053UVT
Connections:
- net CHG_OUT: now also Q1.4 (D), Q2.4 (D)
- net GND: now also Q1.5 (S), Q2.5 (S)
- net HEATER_ON_1: now also Q1.1 (G)
- net HEATER_ON_2: now also Q2.1 (G)
- net at R2.2: now also Q1.3 (G), Q1.6 (D)
- net at R7.2: now also Q2.3 (G), Q2.6 (D)
- net at R3.1, R4.1, R5.1: now also Q1.2 (S)
- net at R10.1, R8.1, R9.1: now also Q2.2 (S)

Commit message: finished routing
Parts:
- R1, R10, R2, R4, R6, R7: footprint (none) -> Resistor_SMD:R_0603_1608Metric
- R3, R5, R8, R9: footprint (none) -> Connector_PinHeader_2.54mm:PinHeader_1x02_P2.54mm_Vertical
Changed lines of the file:
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@@
 			)
 		)
-		(property "Footprint" ""
+		(property "Footprint" "Resistor_SMD:R_0603_1608Metric"
 			(at 115.316 72.644 90)
 			(hide yes)
@@
 			)
 		)
-		(property "Footprint" ""
+		(property "Footprint" "Resistor_SMD:R_0603_1608Metric"
 			(at 91.186 148.844 90)
 			(hide yes)
@@
 			)
 		)
-		(property "Footprint" ""
+		(property "Footprint" "Resistor_SMD:R_0603_1608Metric"
 			(at 141.986 87.884 90)
 			(hide yes)
@@
 			)
 		)
-		(property "Footprint" ""
+		(property "Footprint" "Connector_PinHeader_2.54mm:PinHeader_1x02_P2.54mm_Vertical"
 			(at 116.332 143.51 90)
 			(hide yes)
@@
 			)
 		)
-		(property "Footprint" ""
+		(property "Footprint" "Resistor_SMD:R_0603_1608Metric"
 			(at 91.186 92.964 90)
 			(hide yes)
@@
 			)
 		)
-		(property "Footprint" ""
+		(property "Footprint" "Resistor_SMD:R_0603_1608Metric"
 			(at 115.316 128.524 90)
 			(hide yes)
@@
 			)
 		)
-		(property "Footprint" ""
+		(property "Footprint" "Connector_PinHeader_2.54mm:PinHeader_1x02_P2.54mm_Vertical"
 			(at 127.762 87.63 90)
 			(hide yes)
@@
 			)
 		)
-		(property "Footprint" ""
+		(property "Footprint" "Connector_PinHeader_2.54mm:PinHeader_1x02_P2.54mm_Vertical"
 			(at 116.332 87.63 90)
 			(hide yes)
@@
 			)
 		)
-		(property "Footprint" ""
+		(property "Footprint" "Connector_PinHeader_2.54mm:PinHeader_1x02_P2.54mm_Vertical"
 			(at 127.762 143.51 90)
 			(hide yes)
@@
 			)
 		)
-		(property "Footprint" ""
+		(property "Footprint" "Resistor_SMD:R_0603_1608Metric"
 			(at 141.986 143.764 90)
 			(hide yes)
