File: schematics/connectors.kicad_sch (KiCad schematic)
At the start: 40 parts, among them J1 Conn_01x19, J10 Conn_01x02_Pin, J11 Conn_01x02_Pin, J12 Conn_01x02, J2 Conn_01x06, J3 Conn_01x10, J4 Conn_01x02_Pin, J5 Conn_01x02_Pin, J6 Conn_01x02_Pin, J7 Conn_01x02_Pin, J8 Conn_01x02_Pin, J9 Conn_01x02_Pin

Commit message: Add battery overdischarge & short protections to board
Parts:
- removed BT1, BT2, BT3, BT4, BT5, BT6, BT7, BT8: Battery_Cell, symbol Device:Battery_Cell
- removed J10, J11, J4, J5, J6, J7, J8, J9: Conn_01x02_Pin, Connector_PinSocket_2.54mm:PinSocket_1x02_P2.54mm_Vertical, symbol Connector:Conn_01x02_Pin
- C1, C2, C3, C4: value .1u -> 0.1u
- Rt1, Rt3, Rt5, Rt7: value 15.8k -> 42k
- Rt2, Rt4, Rt6, Rt8: value 5.83k -> 12k
Connections:
- net BATT1- renamed BATT1-P
- net BATT2- renamed BATT2-P
- net BATT3- renamed BATT3-P
- net BATT4- renamed BATT4-P
Other:
- note removed: "actual desired values: 15.7k, 5.78k values are rounded to ones that actually exist"

Commit message: Fix minor issues
Parts:
- Rt1, Rt3, Rt5, Rt7: value 42k -> 11k
- Rt2, Rt4, Rt6, Rt8: value 12k -> 3.9k
Connections:
- net +5V renamed +3V3
